File: docs/prototipo.brd (EAGLE design)
At the start: 68.6 x 53.3 mm, 6 parts

Commit message: Atualização
Parts:
- RRESISTOR 10K ONE: renamed from RRESISTOR ONE
- RRESISTOR 10K THREE: renamed from RRESISTOR TREE
- RRESISTOR 10K TWO: renamed from RRESISTOR TWO
- RRESISTOR 10K ONE: value 230‎Ω -> 10k‎Ω
- RRESISTOR 10K TWO: value 220‎Ω -> 10k‎Ω
Connections:
- removed net N$3 (its old number): RRESISTOR 10K ONE.2, UARDUINO.GND.
- removed net N$4 (its old number): RRESISTOR 10K ONE.1, RRESISTOR 10K TWO.2, UADAPTADOR DE REDE.1
- new net N$8: UADAPTADOR DE REDE.1, UARDUINO.2
- net N$1: now also RRESISTOR 10K ONE.1, UADAPTADOR DE REDE.8, UARDUINO.3.3V; no longer RRESISTOR 10K THREE.2, UADAPTADOR DE REDE.6
- net N$2: now also RRESISTOR 10K TWO.1, UADAPTADOR DE REDE.4, UARDUINO.GND.; no longer RRESISTOR 10K THREE.1, UADAPTADOR DE REDE.8, UARDUINO.3.3V
- net N$5: now also RRESISTOR 10K ONE.2, UADAPTADOR DE REDE.7; no longer RRESISTOR 10K TWO.1, UARDUINO.3
- net N$6: now also RRESISTOR 10K THREE.1, RRESISTOR 10K TWO.2, UADAPTADOR DE REDE.5; no longer UADAPTADOR DE REDE.4, UARDUINO.GND
- net N$7: now also RRESISTOR 10K THREE.2, UARDUINO.3; no longer UADAPTADOR DE REDE.5, UARDUINO.2
Changed lines of the file:
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@@
 </autorouter>
 <elements>
-<element value="" name="UARDUINO" library="AUTODESK_CIRCUITS_BREADBOARD" package="ARDUINO_UNO" x="5" y="10.08"></element><element value="" name="UADAPTADOR DE REDE" library="AUTODESK_CIRCUITS_BREADBOARD" package="2X4P-2.54-65/35MIL" x="5" y="22.78"></element><element value="" name="PIRSENSOR DE MOVIMENTO" library="AUTODESK_CIRCUITS_BREADBOARD" package="1X3P-2.54-2.54-11.6-3.0-BLACK-MALE" x="5" y="35.480000000000004"></element><element value="230‎Ω" name="RRESISTOR ONE" library="AUTODESK_CIRCUITS_BREADBOARD" package="0207/10" x="5" y="48.18"></element><element value="220‎Ω" name="RRESISTOR TWO" library="AUTODESK_CIRCUITS_BREADBOARD" package="0207/10" x="5" y="60.879999999999995"></element><element value="10k‎Ω" name="RRESISTOR TREE" library="AUTODESK_CIRCUITS_BREADBOARD" package="0207/10" x="5" y="73.58"></element></elements>
+<element value="" name="UARDUINO" library="AUTODESK_CIRCUITS_BREADBOARD" package="ARDUINO_UNO" x="5" y="10.08"></element><element value="" name="UADAPTADOR DE REDE" library="AUTODESK_CIRCUITS_BREADBOARD" package="2X4P-2.54-65/35MIL" x="5" y="22.78"></element><element value="" name="PIRSENSOR DE MOVIMENTO" library="AUTODESK_CIRCUITS_BREADBOARD" package="1X3P-2.54-2.54-11.6-3.0-BLACK-MALE" x="5" y="35.480000000000004"></element><element value="10k‎Ω" name="RRESISTOR 10K ONE" library="AUTODESK_CIRCUITS_BREADBOARD" package="0207/10" x="5" y="48.18"></element><element value="10k‎Ω" name="RRESISTOR 10K TWO" library="AUTODESK_CIRCUITS_BREADBOARD" package="0207/10" x="5" y="60.879999999999995"></element><element value="10k‎Ω" name="RRESISTOR 10K THREE" library="AUTODESK_CIRCUITS_BREADBOARD" package="0207/10" x="5" y="73.58"></element></elements>
 <signals>
-<signal name="N$1"><contactref element="RRESISTOR TREE" pad="2"></contactref><contactref element="UADAPTADOR DE REDE" pad="6"></contactref><wire x1="10.08" y1="73.58" x2="6.27" y2="21.51" width="0" layer="19" extent="1-1"></wire></signal><signal name="N$2"><contactref element="RRESISTOR TREE" pad="1"></contactref><contactref element="UARDUINO" pad="3.3V"></contactref><wire x1="-0.08000000000000007" y1="73.58" x2="40.56" y2="12.620000000000001" width="0" layer="19" extent="1-1"></wire><contactref element="UADAPTADOR DE REDE" pad="8"></contactref><wire x1="40.56" y1="12.620000000000001" x2="6.27" y2="26.59" width="0" layer="19" extent="1-1"></wire></signal><signal name="N$3"><contactref element="UARDUINO" pad="GND."></contactref><contactref element="RRESISTOR ONE" pad="2"></contactref><wire x1="48.18" y1="12.620000000000001" x2="10.08" y2="48.18" width="0" layer="19" extent="1-1"></wire></signal><signal name="N$4"><contactref element="UADAPTADOR DE REDE" pad="1"></contactref><contactref element="RRESISTOR ONE" pad="1"></contactref><wire x1="3.73" y1="26.59" x2="-0.08000000000000007" y2="48.18" width="0" layer="19" extent="1-1"></wire><contactref element="RRESISTOR TWO" pad="2"></contactref><wire x1="-0.08000000000000007" y1="48.18" x2="10.08" y2="60.879999999999995" width="0" layer="19" extent="1-1"></wire></signal><signal name="N$5"><contactref element="UARDUINO" pad="3"></contactref><contactref element="RRESISTOR TWO" pad="1"></contactref><wire x1="60.88" y1="60.879999999999995" x2="-0.08000000000000007" y2="60.879999999999995" width="0" layer="19" extent="1-1"></wire></signal><signal name="N$6"><contactref element="UARDUINO" pad="GND"></contactref><contactref element="UADAPTADOR DE REDE" pad="4"></contactref><wire x1="31.416" y1="60.879999999999995" x2="3.73" y2="18.970000000000002" width="0" layer="19" extent="1-1"></wire></signal><signal name="N$7"><contactref element="UADAPTADOR DE REDE" pad="5"></contactref><contactref element="UARDUINO" pad="2"></contactref><wire x1="6.27" y1="18.970000000000002" x2="63.42" y2="60.879999999999995" width="0" layer="19" extent="1-1"></wire></signal><signal name="N$8"><contactref element="PIRSENSOR DE MOVIMENTO" pad="2"></contactref><contactref element="UARDUINO" pad="7"></contactref><wire x1="5" y1="35.480000000000004" x2="50.72" y2="60.879999999999995" width="0" layer="19" extent="1-1"></wire></signal><signal name="N$9"><contactref element="UARDUINO" pad="5V"></contactref><contactref element="PIRSENSOR DE MOVIMENTO" pad="3"></contactref><wire x1="43.1" y1="12.620000000000001" x2="5" y2="32.940000000000005" width="0" layer="19" extent="1-1"></wire></signal><signal name="N$10"><contactref element="PIRSENSOR DE MOVIMENTO" pad="1"></contactref><contactref element="UARDUINO" pad="GND.."></contactref><wire x1="5" y1="38.02" x2="45.64" y2="12.620000000000001" width="0" layer="19" extent="1-1"></wire></signal></signals>
+<signal name="N$1"><contactref element="UARDUINO" pad="3.3V"></contactref><contactref element="RRESISTOR 10K ONE" pad="1"></contactref><wire x1="40.56" y1="12.620000000000001" x2="-0.08000000000000007" y2="48.18" width="0" layer="19" extent="1-1"></wire><contactref element="UADAPTADOR DE REDE" pad="8"></contactref><wire x1="-0.08000000000000007" y1="48.18" x2="6.27" y2="26.59" width="0" layer="19" extent="1-1"></wire></signal><signal name="N$2"><contactref element="UARDUINO" pad="GND."></contactref><contactref element="RRESISTOR 10K TWO" pad="1"></contactref><wire x1="48.18" y1="12.620000000000001" x2="-0.08000000000000007" y2="60.879999999999995" width="0" layer="19" extent="1-1"></wire><contactref element="UADAPTADOR DE REDE" pad="4"></contactref><wire x1="-0.08000000000000007" y1="60.879999999999995" x2="3.73" y2="18.970000000000002" width="0" layer="19" extent="1-1"></wire></signal><signal name="N$3"><contactref element="PIRSENSOR DE MOVIMENTO" pad="1"></contactref><contactref element="UARDUINO" pad="GND.."></contactref><wire x1="5" y1="38.02" x2="45.64" y2="12.620000000000001" width="0" layer="19" extent="1-1"></wire></signal><signal name="N$4"><contactref element="PIRSENSOR DE MOVIMENTO" pad="2"></contactref><contactref element="UARDUINO" pad="7"></contactref><wire x1="5" y1="35.480000000000004" x2="50.72" y2="60.879999999999995" width="0" layer="19" extent="1-1"></wire></signal><signal name="N$5"><contactref element="RRESISTOR 10K ONE" pad="2"></contactref><contactref element="UADAPTADOR DE REDE" pad="7"></contactref><wire x1="10.08" y1="48.18" x2="6.27" y2="24.05" width="0" layer="19" extent="1-1"></wire></signal><signal name="N$6"><contactref element="RRESISTOR 10K TWO" pad="2"></contactref><contactref element="RRESISTOR 10K THREE" pad="1"></contactref><wire x1="10.08" y1="60.879999999999995" x2="-0.08000000000000007" y2="73.58" width="0" layer="19" extent="1-1"></wire><contactref element="UADAPTADOR DE REDE" pad="5"></contactref><wire x1="-0.08000000000000007" y1="73.58" x2="6.27" y2="18.970000000000002" width="0" layer="19" extent="1-1"></wire></signal><signal name="N$7"><contactref element="RRESISTOR 10K THREE" pad="2"></contactref><contactref element="UARDUINO" pad="3"></contactref><wire x1="10.08" y1="73.58" x2="60.88" y2="60.879999999999995" width="0" layer="19" extent="1-1"></wire></signal><signal name="N$8"><contactref element="UADAPTADOR DE REDE" pad="1"></contactref><contactref element="UARDUINO" pad="2"></contactref><wire x1="3.73" y1="26.59" x2="63.42" y2="60.879999999999995" width="0" layer="19" extent="1-1"></wire></signal><signal name="N$9"><contactref element="PIRSENSOR DE MOVIMENTO" pad="3"></contactref><contactref element="UARDUINO" pad="5V"></contactref><wire x1="5" y1="32.940000000000005" x2="43.1" y2="12.620000000000001" width="0" layer="19" extent="1-1"></wire></signal></signals>
 </board>
 </drawing>
